File: HDK/x83-kb.kicad_pcb (KiCad board)
At the start: 2 copper layers, 97 parts, among them U101 AMS1117-3.3, U102 STM32F072RBTx

Commit message: updated pcb
Parts:
- removed C101, C102, C109: 2u2, Capacitor_SMD:C_0805_2012Metric
- removed C103, C104, C105, C106, C107, C108, C110: 100n, Capacitor_SMD:C_0603_1608Metric
- removed R101, R102: 10K, Resistor_SMD:R_0603_1608Metric
- removed U101: AMS1117-3.3, Package_TO_SOT_SMD:SOT-223-3_TabPin2
- removed U102: STM32F072RBTx, Package_QFP:LQFP-64_10x10mm_P0.5mm
- added SW201: ~, x83-kb-lib:SW_OPT_MX, F.Cu at (38.1, 38.1)
- added SW202: ~, x83-kb-lib:SW_OPT_MX, F.Cu at (57.1, 38.1)
- added SW203: ~, x83-kb-lib:SW_OPT_MX, F.Cu at (76.2, 38.1)
- added SW204: ~, x83-kb-lib:SW_OPT_MX, F.Cu at (95.2, 38.1)
- added SW205: ~, x83-kb-lib:SW_OPT_MX, F.Cu at (114.3, 38.1)
- added SW206: ~, x83-kb-lib:SW_OPT_MX, F.Cu at (133.3, 38.1)
- added SW207: ~, x83-kb-lib:SW_OPT_MX, F.Cu at (152.4, 38.1)
- added SW208: ~, x83-kb-lib:SW_OPT_MX, F.Cu at (171.4, 38.1)
- added SW209: ~, x83-kb-lib:SW_OPT_MX, F.Cu at (190.5, 38.1)
- added SW210: ~, x83-kb-lib:SW_OPT_MX, F.Cu at (209.6, 38.1)
- added SW211: ~, x83-kb-lib:SW_OPT_MX, F.Cu at (228.6, 38.1)
- added SW212: ~, x83-kb-lib:SW_OPT_MX, F.Cu at (247.7, 38.1)
- added SW213: ~, x83-kb-lib:SW_OPT_MX, F.Cu at (266.7, 38.1)
- added SW214: ~, x83-kb-lib:SW_OPT_MX, F.Cu at (285.8, 38.1)
- added SW215: ~, x83-kb-lib:SW_OPT_MX, F.Cu at (304.8, 38.1)
- added SW216: ~, x83-kb-lib:SW_OPT_MX, F.Cu at (328.6, 38.1)
- added SW217: ~, x83-kb-lib:SW_OPT_MX, F.Cu at (38.1, 61.9)
- added SW218: ~, x83-kb-lib:SW_OPT_MX, F.Cu at (57.1, 61.9)
- added SW219: ~, x83-kb-lib:SW_OPT_MX, F.Cu at (76.2, 61.9)
- added SW220: ~, x83-kb-lib:SW_OPT_MX, F.Cu at (95.2, 61.9)
- added SW221: ~, x83-kb-lib:SW_OPT_MX, F.Cu at (114.3, 61.9)
- added SW222: ~, x83-kb-lib:SW_OPT_MX, F.Cu at (133.3, 61.9)
- added SW223: ~, x83-kb-lib:SW_OPT_MX, F.Cu at (152.4, 61.9)
- added SW224: ~, x83-kb-lib:SW_OPT_MX, F.Cu at (171.4, 61.9)
- added SW225: ~, x83-kb-lib:SW_OPT_MX, F.Cu at (190.5, 61.9)
- added SW226: ~, x83-kb-lib:SW_OPT_MX, F.Cu at (209.6, 61.9)
- added SW227: ~, x83-kb-lib:SW_OPT_MX, F.Cu at (228.6, 61.9)
- added SW228: ~, x83-kb-lib:SW_OPT_MX, F.Cu at (247.7, 61.9)
- added SW229: ~, x83-kb-lib:SW_OPT_MX, F.Cu at (266.7, 61.9)
- added SW230: ~, x83-kb-lib:SW_OPT_MX, F.Cu at (295.3, 61.9)
- added SW231: ~, x83-kb-lib:SW_OPT_MX, F.Cu at (328.6, 61.9)
- added SW232: ~, x83-kb-lib:SW_OPT_MX, F.Cu at (42.9, 81.0)
- added SW233: ~, x83-kb-lib:SW_OPT_MX, F.Cu at (66.7, 81.0)
- added SW234: ~, x83-kb-lib:SW_OPT_MX, F.Cu at (85.7, 81.0)
- added SW235: ~, x83-kb-lib:SW_OPT_MX, F.Cu at (104.8, 81.0)
- added SW236: ~, x83-kb-lib:SW_OPT_MX, F.Cu at (123.8, 81.0)
- added SW237: ~, x83-kb-lib:SW_OPT_MX, F.Cu at (142.9, 81.0)
- added SW238: ~, x83-kb-lib:SW_OPT_MX, F.Cu at (161.9, 81.0)
- added SW239: ~, x83-kb-lib:SW_OPT_MX, F.Cu at (181.0, 81.0)
- added SW240: ~, x83-kb-lib:SW_OPT_MX, F.Cu at (200.0, 81.0)
- added SW241: ~, x83-kb-lib:SW_OPT_MX, F.Cu at (219.1, 81.0)
- added SW242: ~, x83-kb-lib:SW_OPT_MX, F.Cu at (238.1, 81.0)
- added SW243: ~, x83-kb-lib:SW_OPT_MX, F.Cu at (257.2, 81.0)
- added SW244: ~, x83-kb-lib:SW_OPT_MX, F.Cu at (276.2, 81.0)
- added SW245: ~, x83-kb-lib:SW_OPT_MX, F.Cu at (300.0, 81.0)
- added SW246: ~, x83-kb-lib:SW_OPT_MX, F.Cu at (328.6, 81.0)
- added SW247: ~, x83-kb-lib:SW_OPT_MX, F.Cu at (45.2, 100.0)
- added SW248: ~, x83-kb-lib:SW_OPT_MX, F.Cu at (71.4, 100.0)
- added SW249: ~, x83-kb-lib:SW_OPT_MX, F.Cu at (90.5, 100.0)
- added SW250: ~, x83-kb-lib:SW_OPT_MX, F.Cu at (109.5, 100.0)
- added SW251: ~, x83-kb-lib:SW_OPT_MX, F.Cu at (128.6, 100.0)
- added SW252: ~, x83-kb-lib:SW_OPT_MX, F.Cu at (147.6, 100.0)
- added SW253: ~, x83-kb-lib:SW_OPT_MX, F.Cu at (166.7, 100.0)
- added SW254: ~, x83-kb-lib:SW_OPT_MX, F.Cu at (185.7, 100.0)
- added SW255: ~, x83-kb-lib:SW_OPT_MX, F.Cu at (204.8, 100.0)
- added SW256: ~, x83-kb-lib:SW_OPT_MX, F.Cu at (223.8, 100.0)
- added SW257: ~, x83-kb-lib:SW_OPT_MX, F.Cu at (242.9, 100.0)
- added SW258: ~, x83-kb-lib:SW_OPT_MX, F.Cu at (261.9, 100.0)
- added SW259: ~, x83-kb-lib:SW_OPT_MX, F.Cu at (292.9, 100.0)
- added SW260: ~, x83-kb-lib:SW_OPT_MX, F.Cu at (328.6, 100.0)
- added SW261: ~, x83-kb-lib:SW_OPT_MX, F.Cu at (50.0, 119.1)
- added SW262: ~, x83-kb-lib:SW_OPT_MX, F.Cu at (81.0, 119.1)
- added SW263: ~, x83-kb-lib:SW_OPT_MX, F.Cu at (100.0, 119.1)
- added SW264: ~, x83-kb-lib:SW_OPT_MX, F.Cu at (119.1, 119.1)
- added SW265: ~, x83-kb-lib:SW_OPT_MX, F.Cu at (138.1, 119.1)
- added SW266: ~, x83-kb-lib:SW_OPT_MX, F.Cu at (157.2, 119.1)
- added SW267: ~, x83-kb-lib:SW_OPT_MX, F.Cu at (176.2, 119.1)
- added SW268: ~, x83-kb-lib:SW_OPT_MX, F.Cu at (195.3, 119.1)
- added SW269: ~, x83-kb-lib:SW_OPT_MX, F.Cu at (214.3, 119.1)
- added SW270: ~, x83-kb-lib:SW_OPT_MX, F.Cu at (233.4, 119.1)
- added SW271: ~, x83-kb-lib:SW_OPT_MX, F.Cu at (252.4, 119.1)
- added SW272: ~, x83-kb-lib:SW_OPT_MX, F.Cu at (278.6, 119.1)
- added SW273: ~, x83-kb-lib:SW_OPT_MX, F.Cu at (309.6, 123.8)
- added SW274: ~, x83-kb-lib:SW_OPT_MX, F.Cu at (40.5, 138.1)
- added SW275: ~, x83-kb-lib:SW_OPT_MX, F.Cu at (64.3, 138.1)
- added SW276: ~, x83-kb-lib:SW_OPT_MX, F.Cu at (88.1, 138.1)
- added SW277: ~, x83-kb-lib:SW_OPT_MX, F.Cu at (159.5, 138.1)
- added SW278: ~, x83-kb-lib:SW_OPT_MX, F.Cu at (228.6, 138.1)
- added SW279: ~, x83-kb-lib:SW_OPT_MX, F.Cu at (247.7, 138.1)
- added SW280: ~, x83-kb-lib:SW_OPT_MX, F.Cu at (266.7, 138.1)
- added SW281: ~, x83-kb-lib:SW_OPT_MX, F.Cu at (290.5, 142.9)
- added SW282: ~, x83-kb-lib:SW_OPT_MX, F.Cu at (309.6, 142.9)
- added SW283: ~, x83-kb-lib:SW_OPT_MX, F.Cu at (328.6, 142.9)
- D201, D202, D203, D204, D205, D206, D207, D208, D209, D210, D211, D212, D213, D214, D215, D216, D217, D218, D219, D220, D221, D222, D223, D224, D225, D226, D227, D228, D229, D230, D231, D232, D233, D234, D235, D236, D237, D238, D239, D240, D241, D242, D243, D244, D245, D246, D247, D248, D249, D250, D251, D252, D253, D254, D255, D256, D257, D258, D259, D260, D261, D262, D263, D264, D265, D266, D267, D268, D269, D270, D271, D272, D273, D274, D275, D276, D277, D278, D279, D280, D281, D282, D283: moved to B.Cu
- moved D216 421.0 mm to (338.1, 45.1), turned to 90 degrees
- moved D231 413.4 mm to (338.1, 68.9), turned to 90 degrees
- moved D246 406.3 mm to (338.1, 88.0), turned to 90 degrees
- moved D260 400.4 mm to (338.1, 107.0), turned to 90 degrees
- moved D215 397.2 mm to (314.3, 45.1), turned to 90 degrees
- moved D283 392.7 mm to (338.1, 149.9), turned to 90 degrees
- moved D214 389.9 mm to (295.2, 45.1), turned to 90 degrees
- moved D230 380.4 mm to (304.8, 68.9), turned to 90 degrees
- moved D273 378.7 mm to (319.1, 130.8), turned to 90 degrees
- moved D245 378.3 mm to (309.5, 88.0), turned to 90 degrees
- moved D282 374.5 mm to (319.1, 149.9), turned to 90 degrees
- moved D213 370.4 mm to (276.2, 45.1), turned to 90 degrees
- moved D259 365.8 mm to (302.4, 107.0), turned to 90 degrees
- moved D281 356.6 mm to (300.0, 149.9), turned to 90 degrees
- moved D244 355.2 mm to (285.7, 88.0), turned to 90 degrees
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Connections:
- D201 pad 1: /Keyswitch Matrix/C0 -> /C0
- D202 pad 1: /Keyswitch Matrix/C1 -> /C1
- D203 pad 1: /Keyswitch Matrix/C2 -> /C2
- D204 pad 1: /Keyswitch Matrix/C3 -> /C3
- D205 pad 1: /Keyswitch Matrix/C4 -> /C4
- D206 pad 1: /Keyswitch Matrix/C5 -> /C5
- D207 pad 1: /Keyswitch Matrix/C6 -> /C6
- D208 pad 1: /Keyswitch Matrix/C7 -> /C7
- D209 pad 1: /Keyswitch Matrix/C8 -> /C8
- D210 pad 1: /Keyswitch Matrix/C9 -> /C9
- D211 pad 1: /Keyswitch Matrix/C10 -> /C10
- D212 pad 1: /Keyswitch Matrix/C11 -> /C11
- D213 pad 1: /Keyswitch Matrix/C12 -> /C12
- D214 pad 1: /Keyswitch Matrix/C13 -> /C13
- D215 pad 1: /Keyswitch Matrix/C14 -> /C14
- D216 pad 1: /Keyswitch Matrix/C15 -> /C15
- D217 pad 1: /Keyswitch Matrix/C0 -> /C0
- D218 pad 1: /Keyswitch Matrix/C1 -> /C1
- D219 pad 1: /Keyswitch Matrix/C2 -> /C2
- D220 pad 1: /Keyswitch Matrix/C3 -> /C3
- D221 pad 1: /Keyswitch Matrix/C4 -> /C4
- D222 pad 1: /Keyswitch Matrix/C5 -> /C5
- D223 pad 1: /Keyswitch Matrix/C6 -> /C6
- D224 pad 1: /Keyswitch Matrix/C7 -> /C7
- D225 pad 1: /Keyswitch Matrix/C8 -> /C8
- D226 pad 1: /Keyswitch Matrix/C9 -> /C9
- D227 pad 1: /Keyswitch Matrix/C10 -> /C10
- D228 pad 1: /Keyswitch Matrix/C11 -> /C11
- D229 pad 1: /Keyswitch Matrix/C12 -> /C12
- D230 pad 1: /Keyswitch Matrix/C13 -> /C13
- D231 pad 1: /Keyswitch Matrix/C15 -> /C15
- D232 pad 1: /Keyswitch Matrix/C0 -> /C0
- D233 pad 1: /Keyswitch Matrix/C1 -> /C1
- D234 pad 1: /Keyswitch Matrix/C2 -> /C2
- D235 pad 1: /Keyswitch Matrix/C3 -> /C3
- D236 pad 1: /Keyswitch Matrix/C4 -> /C4
- D237 pad 1: /Keyswitch Matrix/C5 -> /C5
- D238 pad 1: /Keyswitch Matrix/C6 -> /C6
- D239 pad 1: /Keyswitch Matrix/C7 -> /C7
- D240 pad 1: /Keyswitch Matrix/C8 -> /C8
- D241 pad 1: /Keyswitch Matrix/C9 -> /C9
- D242 pad 1: /Keyswitch Matrix/C10 -> /C10
- D243 pad 1: /Keyswitch Matrix/C11 -> /C11
- D244 pad 1: /Keyswitch Matrix/C12 -> /C12
- D245 pad 1: /Keyswitch Matrix/C13 -> /C13
- D246 pad 1: /Keyswitch Matrix/C15 -> /C15
- D247 pad 1: /Keyswitch Matrix/C0 -> /C0
- D248 pad 1: /Keyswitch Matrix/C1 -> /C1
- D249 pad 1: /Keyswitch Matrix/C2 -> /C2
- D250 pad 1: /Keyswitch Matrix/C3 -> /C3
- D251 pad 1: /Keyswitch Matrix/C4 -> /C4
- D252 pad 1: /Keyswitch Matrix/C5 -> /C5
- D253 pad 1: /Keyswitch Matrix/C6 -> /C6
- D254 pad 1: /Keyswitch Matrix/C7 -> /C7
- D255 pad 1: /Keyswitch Matrix/C8 -> /C8
- D256 pad 1: /Keyswitch Matrix/C9 -> /C9
- D257 pad 1: /Keyswitch Matrix/C10 -> /C10
- D258 pad 1: /Keyswitch Matrix/C11 -> /C11
- D259 pad 1: /Keyswitch Matrix/C13 -> /C13
- D260 pad 1: /Keyswitch Matrix/C15 -> /C15
- D261 pad 1: /Keyswitch Matrix/C1 -> /C1
- D262 pad 1: /Keyswitch Matrix/C3 -> /C3
- D263 pad 1: /Keyswitch Matrix/C4 -> /C4
- D264 pad 1: /Keyswitch Matrix/C5 -> /C5
- D265 pad 1: /Keyswitch Matrix/C6 -> /C6
- D266 pad 1: /Keyswitch Matrix/C7 -> /C7
- D267 pad 1: /Keyswitch Matrix/C8 -> /C8
- D268 pad 1: /Keyswitch Matrix/C9 -> /C9
- D269 pad 1: /Keyswitch Matrix/C10 -> /C10
- D270 pad 1: /Keyswitch Matrix/C11 -> /C11
- D271 pad 1: /Keyswitch Matrix/C12 -> /C12
- D272 pad 1: /Keyswitch Matrix/C13 -> /C13
- D273 pad 1: /Keyswitch Matrix/C14 -> /C14
- D274 pad 1: /Keyswitch Matrix/C0 -> /C0
- D275 pad 1: /Keyswitch Matrix/C1 -> /C1
- D276 pad 1: /Keyswitch Matrix/C2 -> /C2
- D277 pad 1: /Keyswitch Matrix/C6 -> /C6
- D278 pad 1: /Keyswitch Matrix/C10 -> /C10
- D279 pad 1: /Keyswitch Matrix/C11 -> /C11
- D280 pad 1: /Keyswitch Matrix/C12 -> /C12
- D281 pad 1: /Keyswitch Matrix/C13 -> /C13
- D282 pad 1: /Keyswitch Matrix/C14 -> /C14
- D283 pad 1: /Keyswitch Matrix/C15 -> /C15
Routing:
- net /C13: track 0.00 -> 83.5 mm
- net /C0: track 0.00 -> 72.3 mm
- net /C1: track 0.00 -> 68.1 mm
- net Net-(D233-A): track 0.00 -> 15.0 mm
- net Net-(D282-A): track 0.00 -> 14.8 mm
- net Net-(D281-A): track 0.00 -> 14.8 mm
- net Net-(D272-A): track 0.00 -> 14.8 mm
- net Net-(D214-A): track 0.00 -> 14.8 mm
- net Net-(D213-A): track 0.00 -> 14.8 mm
- net Net-(D229-A): track 0.00 -> 14.8 mm
- net Net-(D277-A): track 0.00 -> 14.8 mm
- net Net-(D273-A): track 0.00 -> 14.8 mm
- net Net-(D235-A): track 0.00 -> 14.8 mm
- net Net-(D274-A): track 0.00 -> 14.8 mm
- net Net-(D234-A): track 0.00 -> 14.8 mm
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
Commit message: updated pcb
Parts:
- added C101: 2u2, Capacitor_SMD:C_0805_2012Metric, B.Cu at (133.9, 144.9)
- added C102: 2u2, Capacitor_SMD:C_0805_2012Metric, B.Cu at (136.2, 144.9)
- added C103: 100n, Capacitor_SMD:C_0603_1608Metric, B.Cu at (185.8, 149.4)
- added C104: 100n, Capacitor_SMD:C_0603_1608Metric, B.Cu at (188.3, 149.4)
- added C105: 100n, Capacitor_SMD:C_0603_1608Metric, B.Cu at (190.9, 149.4)
- added C106: 100n, Capacitor_SMD:C_0603_1608Metric, B.Cu at (193.4, 149.4)
- added C107: 100n, Capacitor_SMD:C_0603_1608Metric, B.Cu at (195.9, 149.4)
- added C108: 100n, Capacitor_SMD:C_0603_1608Metric, B.Cu at (198.4, 149.4)
- added C109: 2u2, Capacitor_SMD:C_0805_2012Metric, B.Cu at (200.6, 141.1)
- added C110: 100n, Capacitor_SMD:C_0603_1608Metric, B.Cu at (200.9, 149.4)
- added R101: 10K, Resistor_SMD:R_0603_1608Metric, B.Cu at (203.4, 149.4)
- added R102: 10K, Resistor_SMD:R_0603_1608Metric, B.Cu at (205.9, 149.4)
- added REF**: USBC_Receptacle_HRO_TYPE-C-31-M-12, NVF-Kicad:USBC_HRO_TYPE-C-31-M-12, B.Cu at (316.3, 27.4)
- added U101: AMS1117-3.3, Package_TO_SOT_SMD:SOT-223-3_TabPin2, B.Cu at (136.2, 138.6)
- added U102: STM32F072RBTx, Package_QFP:LQFP-64_10x10mm_P0.5mm, B.Cu at (186.4, 137.5)
- moved D282 40.9 mm to (315.2, 109.2), turned to 0 degrees
- moved D283 36.5 mm to (333.3, 113.7), turned to -90 degrees
- moved D281 18.9 mm to (293.2, 132.2), turned to 0 degrees
- moved D273 18.9 mm to (312.2, 113.2), turned to 0 degrees
- moved D238 1.56 mm to (170.3, 86.9)
- moved D243 1.56 mm to (265.6, 86.9)
- moved D244 1.56 mm to (284.6, 86.9)
- moved D245 1.56 mm to (308.4, 86.9)
- moved D246 1.56 mm to (337.0, 86.9)
- moved D254 1.56 mm to (194.1, 105.9)
- moved D258 1.56 mm to (270.3, 105.9)
- moved D259 1.56 mm to (301.3, 105.9)
- moved D260 1.56 mm to (337.0, 105.9)
- moved D275 1.56 mm to (72.7, 144.0)
- moved D276 1.56 mm to (96.5, 144.0)
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Connections:
- D261 pad 1: /C1 -> /C0
- D262 pad 1: /C3 -> /C1
- D263 pad 1: /C4 -> /C2
- D264 pad 1: /C5 -> /C3
- D265 pad 1: /C6 -> /C4
- D266 pad 1: /C7 -> /C5
- D267 pad 1: /C8 -> /C6
- D268 pad 1: /C9 -> /C7
- D269 pad 1: /C10 -> /C8
- D270 pad 1: /C11 -> /C9
- D271 pad 1: /C12 -> /C10
- D272 pad 1: /C13 -> /C12
- D273 pad 1: /C14 -> /C13
- SW202 pad 1: Net-(SW201-A) -> /R0
- SW203 pad 1: Net-(SW202-A) -> /R0
- SW204 pad 1: Net-(SW203-A) -> /R0
- SW205 pad 1: Net-(SW204-A) -> /R0
- SW206 pad 1: Net-(SW205-A) -> /R0
- SW207 pad 1: Net-(SW206-A) -> /R0
- SW208 pad 1: Net-(SW207-A) -> /R0
- SW209 pad 1: Net-(SW208-A) -> /R0
- SW210 pad 1: Net-(SW209-A) -> /R0
- SW211 pad 1: Net-(SW210-A) -> /R0
- SW212 pad 1: Net-(SW211-A) -> /R0
- SW213 pad 1: Net-(SW212-A) -> /R0
- SW214 pad 1: Net-(SW213-A) -> /R0
- SW215 pad 1: Net-(SW214-A) -> /R0
- SW216 pad 1: Net-(SW215-A) -> /R0
- SW218 pad 1: Net-(SW217-A) -> /R1
- SW219 pad 1: Net-(SW218-A) -> /R1
- SW220 pad 1: Net-(SW219-A) -> /R1
- SW221 pad 1: Net-(SW220-A) -> /R1
- SW222 pad 1: Net-(SW221-A) -> /R1
- SW223 pad 1: Net-(SW222-A) -> /R1
- SW224 pad 1: Net-(SW223-A) -> /R1
- SW225 pad 1: Net-(SW224-A) -> /R1
- SW226 pad 1: Net-(SW225-A) -> /R1
- SW227 pad 1: Net-(SW226-A) -> /R1
- SW228 pad 1: Net-(SW227-A) -> /R1
- SW229 pad 1: Net-(SW228-A) -> /R1
- SW230 pad 1: Net-(SW229-A) -> /R1
- SW231 pad 1: Net-(SW230-A) -> /R1
- SW233 pad 1: Net-(SW232-A) -> /R2
- SW234 pad 1: Net-(SW233-A) -> /R2
- SW235 pad 1: Net-(SW234-A) -> /R2
- SW236 pad 1: Net-(SW235-A) -> /R2
- SW237 pad 1: Net-(SW236-A) -> /R2
- SW238 pad 1: Net-(SW237-A) -> /R2
- SW239 pad 1: Net-(SW238-A) -> /R2
- SW240 pad 1: Net-(SW239-A) -> /R2
- SW241 pad 1: Net-(SW240-A) -> /R2
- SW242 pad 1: Net-(SW241-A) -> /R2
- SW243 pad 1: Net-(SW242-A) -> /R2
- SW244 pad 1: Net-(SW243-A) -> /R2
- SW245 pad 1: Net-(SW244-A) -> /R2
- SW246 pad 1: Net-(SW245-A) -> /R2
- SW248 pad 1: Net-(SW247-A) -> /R3
- SW249 pad 1: Net-(SW248-A) -> /R3
- SW250 pad 1: Net-(SW249-A) -> /R3
- SW251 pad 1: Net-(SW250-A) -> /R3
- SW252 pad 1: Net-(SW251-A) -> /R3
- SW253 pad 1: Net-(SW252-A) -> /R3
- SW254 pad 1: Net-(SW253-A) -> /R3
- SW255 pad 1: Net-(SW254-A) -> /R3
- SW256 pad 1: Net-(SW255-A) -> /R3
- SW257 pad 1: Net-(SW256-A) -> /R3
- SW258 pad 1: Net-(SW257-A) -> /R3
- SW259 pad 1: Net-(SW258-A) -> /R3
- SW260 pad 1: Net-(SW259-A) -> /R3
- SW262 pad 1: Net-(SW261-A) -> /R4
- SW263 pad 1: Net-(SW262-A) -> /R4
- SW264 pad 1: Net-(SW263-A) -> /R4
- SW265 pad 1: Net-(SW264-A) -> /R4
- SW266 pad 1: Net-(SW265-A) -> /R4
- SW267 pad 1: Net-(SW266-A) -> /R4
- SW268 pad 1: Net-(SW267-A) -> /R4
- SW269 pad 1: Net-(SW268-A) -> /R4
- SW270 pad 1: Net-(SW269-A) -> /R4
- SW271 pad 1: Net-(SW270-A) -> /R4
- SW272 pad 1: Net-(SW271-A) -> /R4
- SW273 pad 1: Net-(SW272-A) -> /R4
- SW275 pad 1: Net-(SW274-A) -> /R5
- SW276 pad 1: Net-(SW275-A) -> /R5
- SW277 pad 1: Net-(SW276-A) -> /R5
- SW278 pad 1: Net-(SW277-A) -> /R5
- SW279 pad 1: Net-(SW278-A) -> /R5
- SW280 pad 1: Net-(SW279-A) -> /R5
- SW281 pad 1: Net-(SW280-A) -> /R5
- SW282 pad 1: Net-(SW281-A) -> /R5
- SW283 pad 1: Net-(SW282-A) -> /R5
Routing:
- net /R0: track 9.50 -> 442.6 mm
- net /R1: track 9.50 -> 433.1 mm
- net /R2: track 9.50 -> 418.8 mm
- net /R3: track 9.50 -> 416.4 mm
- net /R4: track 9.50 -> 375.6 mm
- net /C15: track 0.00 -> 76.1 mm
- net /C14: track 0.00 -> 67.9 mm
- net /C12: track 0.00 -> 67.5 mm
- net /R5: track 9.50 -> 57.0 mm
- net /C13: track 83.5 -> 121.4 mm
- net Net-(D282-A): track 14.8 -> 39.7 mm
- net Net-(D283-A): track 14.8 -> 31.7 mm
- net Net-(D201-A): track 14.8 -> 0.00 mm
- net Net-(D273-A): track 14.8 -> 4.49 mm
- net Net-(SW271-A): track 9.50 -> 0.00 mm
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Other:
- board outline added: 315 x 130 mm

Commit message: added models
Parts:
- REF**: moved to F.Cu
- turned REF** to 180 degrees
