File: HDK/x83-kb-1.kicad_pcb (KiCad board)
At the start: 2 copper layers, 315 x 130 mm, 180 parts, among them U101 AMS1117-3.3, U102 STM32F072RBTx

Commit message: updated diodes
Parts:
- added REF**: USBC_Receptacle_HRO_TYPE-C-31-M-12, NVF-Kicad:USBC_HRO_TYPE-C-31-M-12, F.Cu at (316.3, 27.4)
- D201, D202, D203, D204, D205, D206, D207, D208, D209, D210, D211, D212, D213, D214, D215, D216, D217, D218, D219, D220, D221, D222, D223, D224, D225, D226, D227, D228, D229, D230, D231, D232, D233, D234, D235, D236, D237, D238, D239, D240, D241, D242, D243, D244, D245, D246, D247, D248, D249, D250, D251, D252, D253, D254, D255, D256, D257, D258, D259, D260, D261, D262, D263, D264, D265, D266, D267, D268, D269, D270, D271, D272, D273, D274, D275, D276, D277, D278, D279, D280, D281, D282, D283: footprint Diode_SMD:D_SOD-123 -> Diode_SMD:D_SMA
- moved D282 43.7 mm to (315.2, 109.2), turned to 0 degrees
- moved D283 39.2 mm to (333.3, 113.7), turned to -90 degrees
- moved D281 20.9 mm to (293.2, 132.2), turned to 0 degrees
- moved D273 20.9 mm to (312.2, 113.2), turned to 0 degrees
- moved D280 4.75 mm to (275.1, 144.0), turned to 90 degrees
- moved D277 4.75 mm to (167.9, 144.0), turned to 90 degrees
- moved D278 4.75 mm to (237.0, 144.0), turned to 90 degrees
- moved D279 4.75 mm to (256.1, 144.0), turned to 90 degrees
- moved D274 4.75 mm to (48.9, 144.0), turned to 90 degrees
- moved D213 4.75 mm to (275.1, 44.0), turned to 90 degrees
- moved D275 4.75 mm to (72.7, 144.0), turned to 90 degrees
- moved D276 4.75 mm to (96.5, 144.0), turned to 90 degrees
- moved D229 4.75 mm to (275.1, 67.8), turned to 90 degrees
- moved D230 4.75 mm to (303.7, 67.8), turned to 90 degrees
- moved D272 4.75 mm to (287.0, 125.0), turned to 90 degrees
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Connections:
- D277 pad 1: /C5 -> /C6
Routing:
- net /R0: track 0.00 -> 442.6 mm
- net /R1: track 0.00 -> 433.1 mm
- net /R2: track 0.00 -> 418.8 mm
- net /R3: track 0.00 -> 416.4 mm
- net /R4: track 0.00 -> 375.6 mm
- net /C14: track 0.00 -> 67.9 mm
- net /R5: track 0.00 -> 57.0 mm
- net /C13: track 68.8 -> 121.4 mm
- net /C2: track 47.8 -> 0.00 mm
- net /C1: track 23.8 -> 68.1 mm
- net /C5: track 43.8 -> 0.00 mm
- net Net-(D282-A): track 7.68 -> 39.7 mm
- net /C15: track 104.8 -> 76.1 mm
- net Net-(D283-A): track 7.68 -> 31.7 mm
- net /C9: track 23.8 -> 0.00 mm
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